File: SolarCellX_v3.sch (KiCad schematic (older format))
At the start: 55 parts, among them J1 XF2M-1015-1A, U2 Value, U3 TSL2561

Commit message: fixed pcb - schematic inconsistencies
Parts:
- C14, C6: footprint Capacitor_SMD:C_0402_1005Metric -> Capacitor_SMD:C_0603_1608Metric
- C9: footprint Capacitor_SMD:C_0603_1608Metric -> Capacitor_SMD:C_0402_1005Metric
- D1: footprint custom-footprints:MICROSMP -> misc-circuits:SOD523
- D2, D3: symbol symbols:MSS1P4-M3_89A -> SolarCellX_v3-rescue:MSS1P4-M3_89A-symbols
- J1: symbol symbols:XF2M-1015-1A -> SolarCellX_v3-rescue:XF2M-1015-1A-symbols
- U2: footprint custom-footprints:NDS8434 -> misc-circuits:QFN50P350X350X100-21N-D
- U3: symbol symbols:TSL2561 -> SolarCellX_v3-rescue:TSL2561-symbols
Connections:
- net VSOLAR: no longer TP4.1
- net VSOLAR_FULL: now reaches D3.2, D4.1 (NEG), SC1.1 (V+), SC2.1 (V+), SC3.1 (V+), SC4.1 (V+)
- net VSOLAR_FULL: now also TP4.1
Changed lines of the file:
@@
 EESchema Schematic File Version 4
 LIBS:SolarCellX_v3-cache
-EELAYER 30 0
+EELAYER 26 0
 EELAYER END
 $Descr A3 16535 11693
@@
 F 0 "D1" H 2650 1819 59  0000 L BNN
 F 1 "SDM20U40-7" H 2400 2059 59  0000 L BNN
-F 2 "custom-footprints:MICROSMP" H 2700 2000 50  0001 C CNN
+F 2 "misc-circuits:SOD523" H 2700 2000 50  0001 C CNN
 F 3 "" H 2700 2000 50  0001 C CNN
 	1    2700 2000
@@
 F 0 "U2" H 5714 2359 69  0000 L BNN
 F 1 "Value" H 5539 2609 69  0001 L BNN
-F 2 "custom-footprints:NDS8434" H 5750 2650 50  0001 C CNN
+F 2 "misc-circuits:QFN50P350X350X100-21N-D" H 5750 2650 50  0001 C CNN
 F 3 "" H 5750 2650 50  0001 C CNN
 	1    5750 2650
@@
 F 0 "C14" H 10108 2661 70  0000 L CNN
 F 1 "100uF" H 10108 2540 70  0000 L CNN
-F 2 "Capacitor_SMD:C_0402_1005Metric" H 10000 2550 50  0001 C CNN
+F 2 "Capacitor_SMD:C_0603_1608Metric" H 10000 2550 50  0001 C CNN
 F 3 "" H 10000 2550 50  0001 C CNN
 	1    10000 2550
@@
 F 0 "C6" H 6958 3161 70  0000 L CNN
 F 1 "100uF" H 6958 3040 70  0000 L CNN
-F 2 "Capacitor_SMD:C_0402_1005Metric" H 6850 3050 50  0001 C CNN
+F 2 "Capacitor_SMD:C_0603_1608Metric" H 6850 3050 50  0001 C CNN
 F 3 "" H 6850 3050 50  0001 C CNN
 	1    6850 3050
@@
 F 0 "C9" H 8158 1961 70  0000 L CNN
 F 1 "0.1uF" H 8158 1840 70  0000 L CNN
-F 2 "Capacitor_SMD:C_0603_1608Metric" H 8050 1850 50  0001 C CNN
+F 2 "Capacitor_SMD:C_0402_1005Metric" H 8050 1850 50  0001 C CNN
 F 3 "" H 8050 1850 50  0001 C CNN
 	1    8050 1850
@@
 	10000 2350 10000 2200
 $Comp
-L symbols:MSS1P4-M3_89A D2
+L SolarCellX_v3-rescue:MSS1P4-M3_89A-symbols D2
 U 1 1 5DC0B0A0
 P 9400 2350
@@
 Flat Flex Connector
 $Comp
-L symbols:XF2M-1015-1A J1
+L SolarCellX_v3-rescue:XF2M-1015-1A-symbols J1
 U 1 1 5DB12088
 P 9100 4600
@@
 SCL1
 $Comp
-L symbols:TSL2561 U3
+L SolarCellX_v3-rescue:TSL2561-symbols U3
 U 1 1 5DB13ECD
 P 9850 5800
@@
 $EndComp
 $Comp
-L symbols:MSS1P4-M3_89A D3
+L SolarCellX_v3-rescue:MSS1P4-M3_89A-symbols D3
 U 1 1 5DC5AC3F
 P 14900 1850
@@
 Text GLabel 7100 6200 3    50   Output ~ 0
 VBAT
-Text GLabel 7350 6200 3    50   BiDi ~ 0
-VSOLAR
 Text Notes 6650 5900 0    100  ~ 0
 Test Points
+Text Label 14550 1450 0    50   ~ 0
+VSOLAR_FULL
+Text Label 7350 6350 0    50   ~ 0
+VSOLAR_FULL
+Wire Wire Line
+	7350 6200 7350 6350
 $EndSCHEMATC

Commit message: moved solar panel and sun sensor. Fixed PCB design rules
Parts:
- D2, D3: footprint custom-footprints:MICROSMP -> misc-circuits:MICROSMP
Changed lines of the file:
@@
 F 0 "D2" H 9700 2085 50  0000 C CNN
 F 1 "MSS1P4-M3_89A" H 9700 2176 50  0000 C CNN
-F 2 "custom-footprints:MICROSMP" H 9800 2500 50  0001 L BNN
+F 2 "misc-circuits:MICROSMP" H 9800 2500 50  0001 L BNN
 F 3 "https://www.vishay.com/docs/89019/mss1p4.pdf" H 9800 2400 50  0001 L BNN
 F 4 "Vishay MSS1P4-M3/89A SMT Schottky Diode, 40V 1A, 2-Pin uSMP" H 9800 2300 50  0001 L BNN "Description"
@@
 F 0 "D3" H 15200 1585 50  0000 C CNN
 F 1 "MSS1P4-M3_89A" H 15200 1676 50  0000 C CNN
-F 2 "custom-footprints:MICROSMP" H 15300 2000 50  0001 L BNN
+F 2 "misc-circuits:MICROSMP" H 15300 2000 50  0001 L BNN
 F 3 "https://www.vishay.com/docs/89019/mss1p4.pdf" H 15300 1900 50  0001 L BNN
 F 4 "Vishay MSS1P4-M3/89A SMT Schottky Diode, 40V 1A, 2-Pin uSMP" H 15300 1800 50  0001 L BNN "Description"
